File: PCB/MkI/MkI.kicad_sch (KiCad schematic)
At the start: 13 parts, among them J1 Conn_RX, J2 Conn_TX, U1 CH32V003FxPx

Commit message: MkI PCB Finished
Parts:
- removed TP1: GND, symbol Connector:TestPoint
- removed TP3: VCC, symbol Connector:TestPoint
- added Q1, Q2, Q3: AO3400A, Project_Footprints:SOT-23_Clean, symbol Transistor_FET:AO3400A
- added R1: 10R, Resistor_SMD:R_0603_1608Metric, symbol Device:R
- added R2: 2K2, Resistor_SMD:R_0603_1608Metric, symbol Device:R
- TP1: renamed from TP2; footprint (none) -> TestPoint:TestPoint_Pad_D1.0mm
Connections:
- net GND: now also Q1.2 (S), Q2.2 (S), Q3.2 (S)
- net GPIO_PD7: now also R1.1
- net VCC: now also R2.2
- net DIGIT_2: now reaches DISP1.11 (DIGIT_2)
- net DIGIT_2: now also Q2.3 (D)
- net DIGIT_1: now reaches DISP1.16 (DIGIT_1)
- net DIGIT_1: now also Q1.3 (D)
- new net: Q1.1 (G), Q3.3 (D), R2.1
- new net: Q2.1 (G), Q3.1 (G), R1.2
Other:
- note added: "Daisychain Connectors"
- note added: "Display Digit Inverter"
- note removed: "Daisy Chain Connectors"
- moved on the sheet: DISP1, RN1, RN2, RN3, RN4, TP1

Commit message: Added Images
Other:
- title: (none) -> 00314S2D-ASCII
Changed lines of the file:
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@@
 	(generator_version "8.0")
 	(paper "A4")
+	(title_block
+		(title "00314S2D-ASCII")
+		(date "2024-09-15")
+		(rev "MkI")
+	)
 	(junction
 		(at 106.045 36.195)

Commit message: Changed current limiting resistors
Parts:
- RN1, RN2, RN3, RN4: value 150R -> 330R
Other:
- moved on the sheet: C1, C2, J1, J2, TP1, U1
